File: circuts/moonlight.sch (KiCad schematic (older format))
At the start: 9 parts, among them IC1 ATTINY45-P, P1 CONN_4, P2 V12, Q1 MOSFET_N, Q2 MOSFET_N, Q3 MOSFET_N, SW1 SW_PUSH, SW2 SW_PUSH, U1 78L05

Commit message: Added PCB board.
Parts:
- added C1: CP1, symbol CP1
Connections:
- net GND: now also C1.2
- net at Q1.G: now also IC1.5 (PB0(MOSI/DI/SDA/AIN0/OC0A/OC1A/AREF/PCINT0)); no longer IC1.7 (PB2(SCK/USCK/SCL/T0/INT0/ADC1/PCINT2))
- net at Q3.G: now also IC1.7 (PB2(SCK/USCK/SCL/T0/INT0/ADC1/PCINT2)); no longer IC1.5 (PB0(MOSI/DI/SDA/AIN0/OC0A/OC1A/AREF/PCINT0))
- net at IC1.8 (VCC), U1.VO: now also C1.1
Changed lines of the file:
@@
-EESchema Schematic File Version 2  date Сб. 09 февр. 2013 00:02:51
+EESchema Schematic File Version 2  date Сб. 09 февр. 2013 00:36:02
 LIBS:power
 LIBS:device
@@
 LIBS:contrib
 LIBS:valves
-EELAYER 43  0
+LIBS:moonlight-cache
+EELAYER 25  0
 EELAYER END
 $Descr A4 11700 8267
@@
 Comment4 ""
 $EndDescr
+Connection ~ 6650 3600
+Wire Wire Line
+	6650 3550 6650 3700
+Wire Wire Line
+	3950 2250 3950 2700
+Wire Wire Line
+	3950 2700 3700 2700
+Wire Wire Line
+	3700 2700 3700 3300
+Wire Wire Line
+	3700 3300 3850 3300
+Wire Wire Line
+	3350 3200 3350 3100
+Wire Wire Line
+	3350 3100 3850 3100
+Wire Wire Line
+	3650 2450 2550 2450
+Wire Wire Line
+	3500 2100 3500 2050
+Wire Wire Line
+	5600 1950 5600 2050
+Wire Wire Line
+	2400 3000 2600 3000
+Wire Wire Line
+	2600 3000 2600 3400
+Wire Wire Line
+	2600 3400 3050 3400
+Wire Wire Line
+	2400 2800 2550 2800
+Wire Wire Line
+	3050 2550 3050 2500
+Wire Wire Line
+	3050 2500 3200 2500
+Wire Wire Line
+	2400 2700 2450 2700
+Wire Wire Line
+	2450 2700 2450 2500
+Wire Wire Line
+	8050 2800 8050 3100
+Wire Wire Line
+	3000 4000 3000 3950
+Wire Wire Line
+	3000 3950 3050 3950
+Wire Wire Line
+	3650 3700 3650 3400
+Wire Wire Line
+	3650 3400 3850 3400
+Wire Wire Line
+	8000 3500 8000 3300
+Wire Wire Line
+	8000 3300 8100 3300
+Wire Wire Line
+	6650 3600 6550 3600
+Wire Wire Line
+	6800 3100 6550 3100
+Wire Wire Line
+	7200 2800 7200 2650
+Wire Wire Line
+	7200 2650 7500 2650
+Wire Wire Line
+	7500 2650 7500 2700
+Wire Wire Line
+	8100 3100 7600 3100
+Wire Wire Line
+	3850 3500 3750 3500
+Wire Wire Line
+	3750 3500 3750 3950
+Wire Wire Line
+	3750 3950 3650 3950
+Wire Wire Line
+	3050 3700 3000 3700
+Wire Wire Line
+	3000 3700 3000 3750
+Connection ~ 8050 3100
+Wire Wire Line
+	3050 3000 2900 3000
+Wire Wire Line
+	2900 3000 2900 3100
+Wire Wire Line
+	3200 2900 2400 2900
+Wire Wire Line
+	5250 1950 5250 2050
+Wire Wire Line
+	3500 2050 3650 2050
 Wire Wire Line
 	2550 2800 2550 2450
 Wire Wire Line
-	3650 2050 3500 2050
-Wire Wire Line
-	5250 1950 5250 2050
-Wire Wire Line
-	3200 2900 2400 2900
-Wire Wire Line
-	2900 3100 2900 3000
-Wire Wire Line
-	2900 3000 3050 3000
-Wire Wire Line
-	3850 3100 3850 2850
-Wire Wire Line
-	3850 2850 3950 2850
-Wire Wire Line
-	3950 2850 3950 2250
-Wire Wire Line
-	3500 2700 3600 2700
-Wire Wire Line
-	3600 2700 3600 3200
-Wire Wire Line
-	3350 3200 3450 3200
-Wire Wire Line
-	3450 3200 3450 3300
-Connection ~ 8050 3100
-Wire Wire Line
-	3000 3750 3000 3700
-Wire Wire Line
-	3000 3700 3050 3700
-Wire Wire Line
-	3650 3950 3750 3950
-Wire Wire Line
-	3750 3950 3750 3500
-Wire Wire Line
-	3750 3500 3850 3500
-Wire Wire Line
-	8100 3100 7600 3100
-Wire Wire Line
-	7500 2700 7500 2650
-Wire Wire Line
-	7500 2650 7200 2650
-Wire Wire Line
-	7200 2650 7200 2800
-Wire Wire Line
-	6800 3100 6550 3100
-Wire Wire Line
-	6550 3600 6650 3600
-Wire Wire Line
-	6650 3600 6650 3700
-Wire Wire Line
-	8100 3300 8000 3300
-Wire Wire Line
-	8000 3300 8000 3500
-Wire Wire Line
-	3850 3400 3650 3400
-Wire Wire Line
-	3650 3400 3650 3700
-Wire Wire Line
-	3050 3950 3000 3950
-Wire Wire Line
-	3000 3950 3000 4000
-Wire Wire Line
-	8050 2800 8050 3100
-Wire Wire Line
-	3450 3300 3850 3300
-Wire Wire Line
-	3600 3200 3850 3200
-Wire Wire Line
-	2450 2500 2450 2700
-Wire Wire Line
-	2450 2700 2400 2700
-Wire Wire Line
-	3200 2500 3050 2500
-Wire Wire Line
-	3050 2500 3050 2550
-Wire Wire Line
-	2550 2800 2400 2800
-Wire Wire Line
-	3050 3400 2600 3400
-Wire Wire Line
-	2600 3400 2600 3000
-Wire Wire Line
-	2600 3000 2400 3000
-Wire Wire Line
-	5600 1950 5600 2050
-Wire Wire Line
-	3500 2050 3500 2100
-Wire Wire Line
-	2550 2450 3650 2450
-$Comp
-L +12V #PWR01
+	3850 3200 3500 3200
+Wire Wire Line
+	3500 3200 3500 2700
+Wire Wire Line
+	6650 3100 6650 3150
+Connection ~ 6650 3100
+$Comp
+L CP1 C1
+U 1 1 5115619F
+P 6650 3350
+F 0 "C1" H 6700 3450 50  0000 L CNN
+F 1 "CP1" H 6700 3250 50  0000 L CNN
+	1    6650 3350
+	1    0    0    -1
+$EndComp
+$Comp
+L +12V #PWR8
 U 1 1 51155936
 P 5600 2050
-F 0 "#PWR01" H 5600 2000 20  0001 C CNN
+F 0 "#PWR8" H 5600 2000 20  0001 C CNN
 F 1 "+12V" H 5600 2150 30  0000 C CNN
 	1    5600 2050
@@
 $EndComp
 $Comp
-L GND #PWR02
+L GND #PWR7
 U 1 1 51155933
 P 5250 2050
-F 0 "#PWR02" H 5250 2050 30  0001 C CNN
+F 0 "#PWR7" H 5250 2050 30  0001 C CNN
 F 1 "GND" H 5250 1980 30  0001 C CNN
 	1    5250 2050
@@
 $EndComp
 $Comp
-L PWR_FLAG #FLG03
+L PWR_FLAG #FLG2
 U 1 1 51155930
 P 5600 1950
-F 0 "#FLG03" H 5600 2045 30  0001 C CNN
+F 0 "#FLG2" H 5600 2045 30  0001 C CNN
 F 1 "PWR_FLAG" H 5600 2130 30  0000 C CNN
 	1    5600 1950
@@
 $EndComp
 $Comp
-L PWR_FLAG #FLG04
+L PWR_FLAG #FLG1
 U 1 1 511559B8
 P 5250 1950
-F 0 "#FLG04" H 5250 2045 30  0001 C CNN
+F 0 "#FLG1" H 5250 2045 30  0001 C CNN
 F 1 "PWR_FLAG" H 5250 2130 30  0000 C CNN
 	1    5250 1950
@@
 $EndComp
 $Comp
-L GND #PWR05
+L GND #PWR6
 U 1 1 511557E0
 P 3500 2100
-F 0 "#PWR05" H 3500 2100 30  0001 C CNN
+F 0 "#PWR6" H 3500 2100 30  0001 C CNN
 F 1 "GND" H 3500 2030 30  0001 C CNN
 	1    3500 2100
@@
 $EndComp
 $Comp
-L GND #PWR06
+L GND #PWR5
 U 1 1 511557DE
 P 3050 2550
-F 0 "#PWR06" H 3050 2550 30  0001 C CNN
+F 0 "#PWR5" H 3050 2550 30  0001 C CNN
 F 1 "GND" H 3050 2480 30  0001 C CNN
 	1    3050 2550
@@
 $EndComp
 $Comp
-L GND #PWR07
+L GND #PWR2
 U 1 1 511557DD
 P 2900 3100
-F 0 "#PWR07" H 2900 3100 30  0001 C CNN
+F 0 "#PWR2" H 2900 3100 30  0001 C CNN
 F 1 "GND" H 2900 3030 30  0001 C CNN
 	1    2900 3100
@@
 $EndComp
 $Comp
-L +12V #PWR08
+L +12V #PWR1
 U 1 1 511557BF
 P 2450 2500
-F 0 "#PWR08" H 2450 2450 20  0001 C CNN
+F 0 "#PWR1" H 2450 2450 20  0001 C CNN
 F 1 "+12V" H 2450 2600 30  0000 C CNN
 	1    2450 2500
@@
 $EndComp
 $Comp
-L +12V #PWR09
+L +12V #PWR12
 U 1 1 51155918
 P 8050 2800
-F 0 "#PWR09" H 8050 2750 20  0001 C CNN
+F 0 "#PWR12" H 8050 2750 20  0001 C CNN
 F 1 "+12V" H 8050 2900 30  0000 C CNN
 	1    8050 2800
@@
 $EndComp
 $Comp
-L GND #PWR010
+L GND #PWR3
 U 1 1 511552F7
 P 3000 3750
-F 0 "#PWR010" H 3000 3750 30  0001 C CNN
+F 0 "#PWR3" H 3000 3750 30  0001 C CNN
 F 1 "GND" H 3000 3680 30  0001 C CNN
 	1    3000 3750
@@
 $EndComp
 $Comp
-L GND #PWR011
+L GND #PWR4
 U 1 1 511552F3
 P 3000 4000
-F 0 "#PWR011" H 3000 4000 30  0001 C CNN
+F 0 "#PWR4" H 3000 4000 30  0001 C CNN
 F 1 "GND" H 3000 3930 30  0001 C CNN
 	1    3000 4000
@@
 $EndComp
 $Comp
-L GND #PWR012
+L GND #PWR11
 U 1 1 51155202
 P 8000 3500
-F 0 "#PWR012" H 8000 3500 30  0001 C CNN
+F 0 "#PWR11" H 8000 3500 30  0001 C CNN
 F 1 "GND" H 8000 3430 30  0001 C CNN
 	1    8000 3500
@@
 $EndComp
 $Comp
-L GND #PWR013
+L GND #PWR9
 U 1 1 511551F1
 P 6650 3700
-F 0 "#PWR013" H 6650 3700 30  0001 C CNN
+F 0 "#PWR9" H 6650 3700 30  0001 C CNN
 F 1 "GND" H 6650 3630 30  0001 C CNN
 	1    6650 3700
@@
 $EndComp
 $Comp
-L GND #PWR014
+L GND #PWR10
 U 1 1 51155915
 P 7500 2700
-F 0 "#PWR014" H 7500 2700 30  0001 C CNN
+F 0 "#PWR10" H 7500 2700 30  0001 C CNN
 F 1 "GND" H 7500 2630 30  0001 C CNN
 	1    7500 2700
